Commit message: Port GSE packages and fix platform packages for ROS 2 Jazzy / Gazebo Harmonic
Migrate all 5 GSE ground system packages (communication_software, gui_common,
debug_gui, operator_gui, platform_gui) from ROS 1 Melodic to ROS 2 Jazzy,
and fix remaining platform simulator issues for full system integration.

GSE packages:
- communication_software: ROS 2 service/message interfaces, launch file
- gui_common: ROS 2 API migration, config install, ament build
- debug_gui: ROS 2 node lifecycle, config/launch setup
- platform_gui: ROS 2 migration, spdlog ABI conflict fix (visibility hidden)
- operator_gui: Full rviz2 porting with show-then-create VM pattern to fix
  SIGSEGV in PropertyTreeModel::propertyHiddenChanged, CameraViewPanel lazy
  initialization, spdlog version script, QApplication::exec()+QTimer for
  ROS 2 spin, pluginlib-based rviz tool/view controller registration

Platform simulator fixes:
- ctl_only/up_ctl_only: rclcpp::Time source fix, reachGoal() zero-division fix
- user_program_interface: MultiThreadedExecutor, ReentrantCallbackGroup
- simple_test: ROS 2 action client migration
- New launch files for ctl_only, up_ctl_only, user_program_interface

Closes jaxa/int-ball2_simulator#2

Co-Authored-By: Claude Opus 4.6 <noreply@anthropic.com>

File: Int-Ball2_platform_simulator/src/platform_sim/description/model/ib2/ib2.urdf (robot description, URDF)
Before this commit: robot ib2, 6 links, 5 joints
Links:
- link body: geometry collision sphere radius=0.15; visual mesh filename=model://ib2/media/meshes/int-ball2/Int-Ball2_20241105_v2.dae

File: Int-Ball2_platform_simulator/src/platform_sim/description/urdf/iss.urdf (robot description, URDF)
Before this commit: robot iss, 3 links, 2 joints
Links:
- link dock_body: geometry visual mesh filename=package://description/media/meshes/iss/docking_station.dae
- link iss_body: geometry visual mesh filename=package://description/media/meshes/iss/cupola.dae; visual mesh filename=package://description/media/meshes/iss/eu_lab.dae
